File: RGB-Pixel/rgb3-panelized2.brd (EAGLE design)
At the start: 17.8 x 10.2 mm, 3 parts, among them X1 MICROMATCH-4, X2 MICROMATCH-4

Commit message: added reversed files
Parts:
- flipped X1 to the bottom, turned to 90 degrees
- flipped X2 to the bottom
Routing:
- net N$4: track 22.1 -> 17.6 mm
- net N$1: track 26.2 -> 22.3 mm
- net N$6: track 5.66 -> 3.12 mm
- net N$5: track 2.94 -> 5.48 mm
- net N$3: track 3.73 -> 2.94 mm
Other:
- board text added: "LED1"
- board text added: "X1"
- board text added: "X2"
